File: WaccaTouchPanel-pcb/WaccaTouchPanel.kicad_pcb (KiCad board)
At the start: 2 copper layers, 254.9 x 231.1 mm, 106 parts, among them IC1 W25Q16JVUXIQ_TR, IC2 AT42QT2120-MMHR, IC3 AT42QT2120-MMHR, J1 USB_C_Receptacle_USB2.0, J10 SESNSOR2, J11 SESNSOR9, J12 SESNSOR1, J13 SESNSOR10, J14 SESNSOR11, J15 SESNSOR12, J16 SESNSOR19, J17 SESNSOR18, J18 SESNSOR17, J19 SESNSOR16, J2 RJ45_LED_Shielded, J20 SESNSOR15, J21 SESNSOR20, J22 SESNSOR14, J23 SESNSOR13, J24 Conn_02x06_Odd_Even, J25 Conn_02x06_Odd_Even, J26 Conn_02x06_Odd_Even, J27 Conn_02x06_Odd_Even, J28 Conn_02x06_Odd_Even, J3 SESNSOR7, J4 SESNSOR6, J5 Conn_01x03_Male, J6 SESNSOR5, J7 SESNSOR4, J8 SESNSOR3, J9 SESNSOR8, SW1 Program, SW3 Reset, U1 NCP1117-3.3_SOT223, U3 RP2040, Y1 ABLS-12.000MHZ-B4-T

Commit message: finished Touch Panel PCB and added it to actions
Parts:
- removed J24, J25, J26, J27, J28: Conn_02x06_Odd_Even, Connector_PinHeader_2.54mm:PinHeader_2x06_P2.54mm_Vertical
Connections:
- D10 pad 4: LED_C2_R3_I -> LED_C2_R2_O
- D11 pad 4: LED_C2_R4_I -> LED_C2_R3_O
- D12 pad 2: LED_C2_R5_O -> LED_C2_R6_I
- D12 pad 4: LED_C2_R5_I -> LED_C2_R4_O
- D14 pad 4: LED_C3_R2_I -> LED_C3_R1_O
- D15 pad 4: LED_C3_R3_I -> LED_C3_R2_O
- D16 pad 4: LED_C3_R4_I -> LED_C3_R3_O
- D17 pad 4: LED_C3_R5_I -> LED_C3_R4_O
- D18 pad 2: LED_C4_R1_O -> LED_C4_R2_I
- D18 pad 4: LED_C4_R1_I -> LED_C5_R8_O
- D19 pad 2: LED_C4_R2_O -> LED_C4_R3_I
- D20 pad 2: LED_C4_R3_O -> LED_C4_R4_I
- D21 pad 2: LED_C4_R4_O -> LED_C4_R5_I
- D23 pad 2: LED_C5_R1_O -> LED_C5_R2_I
- D24 pad 2: LED_C5_R2_O -> LED_C5_R3_I
- D25 pad 2: LED_C5_R3_O -> LED_C5_R4_I
- D26 pad 2: LED_C5_R4_O -> LED_C5_R5_I
- D28 pad 4: LED_C1_R6_I -> LED_C1_R5_O
- D29 pad 4: LED_C1_R7_I -> LED_C1_R6_O
- D30 pad 4: LED_C1_R8_I -> LED_C1_R7_O
- D32 pad 4: LED_C2_R7_I -> LED_C2_R6_O
- D33 pad 2: LED_C2_R8_O -> LED_C1_R1_I
- D33 pad 4: LED_C2_R8_I -> LED_C2_R7_O
- D34 pad 4: LED_C3_R6_I -> LED_C3_R5_O
- D35 pad 4: LED_C3_R7_I -> LED_C3_R6_O
- D36 pad 4: LED_C3_R8_I -> LED_C3_R7_O
- D37 pad 4: LED_C4_R6_I -> LED_C4_R5_O
- D38 pad 4: LED_C4_R7_I -> LED_C4_R6_O
- D39 pad 2: LED_C4_R8_O -> LED_C3_R1_I
- D39 pad 4: LED_C4_R8_I -> LED_C4_R7_O
- D4 pad 4: LED_C1_R2_I -> LED_C1_R1_O
- D40 pad 4: LED_C5_R6_I -> LED_C5_R5_O
- D41 pad 4: LED_C5_R7_I -> LED_C5_R6_O
- D42 pad 4: LED_C5_R8_I -> LED_C5_R7_O
- D5 pad 4: LED_C1_R3_I -> LED_C1_R2_O
- D6 pad 4: LED_C1_R4_I -> LED_C1_R3_O
- D7 pad 4: LED_C1_R5_I -> LED_C1_R4_O
- D8 pad 4: LED_C2_R1_I -> LED_C3_R8_O
- D9 pad 4: LED_C2_R2_I -> LED_C2_R1_O
- J2 pad 2: LED_OUT -> LED_C1_R8_O
- J2 pad 4: LED_IN -> LED_C5_R1_I
Routing:
- net VCC_IN: track 95.1 -> 1896.4 mm, vias 0 -> 7
- net Earth: track 360.4 -> 2073.1 mm, vias 1 -> 41
- net LED_C5_R8_O: track 0.00 -> 253.4 mm
- net LED_C3_R1_I: track 0.00 -> 249.3 mm, vias 0 -> 2
- net LED_C3_R8_O: track 0.00 -> 240.5 mm
- net LED_C1_R1_I: track 0.00 -> 231.6 mm
- net LED_C1_R8_O: track 0.00 -> 219.7 mm, vias 0 -> 2
- net +3.3V: track 80.1 -> 238.8 mm, vias 3 -> 6
- net LED_C5_R1_I: track 0.00 -> 146.5 mm, vias 0 -> 1
- net Net-(IC3-Pad6): track 0.00 -> 121.4 mm
- net Net-(IC3-Pad5): track 225.4 -> 103.9 mm
- net Net-(IC2-Pad20): track 168.4 -> 90.1 mm
- net Net-(IC2-Pad1): track 0.00 -> 78.3 mm
- net Net-(IC2-Pad5): track 138.6 -> 62.4 mm
- net Net-(IC2-Pad6): track 0.00 -> 76.2 mm
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