File: WaccaProtocolTranslator-pcb/WaccaProtocolTranslator.kicad_sch (KiCad schematic)
At the start: 104 parts

Commit message: designed the Protocol Translator PCB and added a PCB build task during production file generation
Parts:
- removed J? (x12): RJ45_LED_Shielded, symbol Connector:RJ45_LED_Shielded
- removed J?: Screw_Terminal_01x02, symbol Connector:Screw_Terminal_01x02
- removed J?: Conn_02x13_Odd_Even, symbol Connector_Generic:Conn_02x13_Odd_Even
- removed R? (x21): 150, symbol Device:R_US
- added C13, C19: 0.1u, Capacitor_SMD:C_0402_1005Metric, symbol Device:C_Small
- added C23, C24: 10u, Capacitor_SMD:C_0402_1005Metric, symbol Device:C_Small
- added C30, C31: 27p, Capacitor_SMD:C_0402_1005Metric, symbol Device:C_Small
- added D1: B320, Diode_SMD:D_SMC, symbol Diode:B320
- added J10, J9: Barrel_Jack, Connector_BarrelJack:BarrelJack_CUI_PJ-063AH_Horizontal, symbol Connector:Barrel_Jack
- added J4: USB_C_Receptacle_USB2.0, Connector_USB:USB_C_Receptacle_Amphenol_12401548E4-2A, symbol Connector:USB_C_Receptacle_USB2.0
- added J7: Conn_02x02_Odd_Even, Connector_PinHeader_2.54mm:PinHeader_2x02_P2.54mm_Vertical, symbol Connector_Generic:Conn_02x02_Odd_Even
- added J8: Conn_01x08_Male, Connector_PinHeader_2.54mm:PinHeader_1x08_P2.54mm_Vertical, symbol Connector:Conn_01x08_Male
- added Q1, Q2: IRLB8721PBF, SamacSys_Parts:TO254P483X1016X1994-3P, symbol SamacSys_Parts:IRLB8721PBF
- added R10, R9: 5K1, Resistor_SMD:R_0402_1005Metric, symbol Device:R_US
- added R12: 3.3K, Resistor_SMD:R_0402_1005Metric, symbol Device:R_US
- added R14, R8: 2.2K, Resistor_SMD:R_0402_1005Metric, symbol Device:R_US
- added R16, R17, R18, R19, R20, R21, R22, R23, R24, R25, R26, R36, R37, R38, R39, R40, R41, R42, R43, R44, R45: 150, Resistor_SMD:R_0402_1005Metric, symbol Device:R_US
- added R46, R47: 275, Resistor_SMD:R_0402_1005Metric, symbol Device:R_US
- added U2: 93LCxxB, SamacSys_Parts:SOP65P490X110-8N, symbol Memory_EEPROM:93LCxxB
- added U4: FT232HQ-REEL, SamacSys_Parts:QFN50P800X800X100-49N-D, symbol SamacSys_Parts:FT232HQ-REEL
- added Y3: ABLS-12.000MHZ-B4-T, Crystal:Crystal_HC49-4H_Vertical, symbol Device:Crystal
- C1, C10, C11, C12, C14, C15, C16, C17, C18, C2, C20, C21, C22, C25, C26, C27, C28, C29, C3, C32, C33, C34, C35, C36, C37, C38, C39, C4, C5, C6, C7, C8, C9: renamed from C?; footprint (none) -> Capacitor_SMD:C_0402_1005Metric
- IC1, IC2: renamed from IC?; footprint SON50P300X200X60-9N -> SamacSys_Parts:SON50P300X200X60-9N
- J1, J3: renamed from J?; footprint (none) -> Connector_USB:USB_C_Receptacle_Amphenol_12401548E4-2A
- J2: renamed from J?; footprint 61163141 -> SamacSys_Parts:61163141
- J5, J6: renamed from J?; footprint (none) -> Connector_PinHeader_2.54mm:PinHeader_1x03_P2.54mm_Vertical
- R1, R11, R13, R15, R2, R3, R31, R32, R33, R34, R35, R4, R5, R6, R7: renamed from R?; footprint (none) -> Resistor_SMD:R_0402_1005Metric
- R27, R28, R29, R30: renamed from R?; value 500 -> 2.2K; footprint (none) -> Resistor_SMD:R_0402_1005Metric
- SW1, SW2, SW3: renamed from SW?; footprint (none) -> Button_Switch_SMD:SW_SPST_B3U-1000P
- Y1, Y2: renamed from Y?; footprint RP2040_minimal:Crystal_SMD_HC49-US -> Crystal:Crystal_HC49-4H_Vertical
- gave numbers to parts that had none: 5
Connections:
- net TP1_LL is gone; now on net TPL1_LL: R15.2
- net TP7_LL is gone; now on net TPR1_LL: R34.2
- net TP7_RL is gone; now on net TPR1_RL: R35.2
- net Earth: now also J2.A10 (K_GREEN_1), J2.A12 (K_GREEN_2), J2.B10 (K_GREEN_3), J2.B12 (K_GREEN_4), J2.C10 (K_GREEN_5), J2.C12 (K_GREEN_6), J2.D10 (K_GREEN_7), J2.D12 (K_GREEN_8), J2.E10 (K_GREEN_9), J2.E12 (K_GREEN_10), J2.F10 (K_GREEN_11), J2.F12 (K_GREEN_12), J2.G11 (K_GREEN_14), J2.G9 (K_GREEN_13), J2.H11 (K_GREEN_16), J2.H9 (K_GREEN_15), J2.J11 (K_GREEN_18), J2.J9 (K_GREEN_17), J2.K11 (K_GREEN_20), J2.K9 (K_GREEN_19), J2.L11 (K_GREEN_22), J2.L9 (K_GREEN_21), J2.M11 (K_GREEN_24), J2.M9 (K_GREEN_23), J2.MH1 (MH3), J2.MH2 (MH8), J2.MH3 (MH7), J2.MH4 (MH6), J2.MH5, J2.MH6 (MH4), C13.2, C19.1, C23.2, C24.2, C30.1, C31.1, J10.2, J4.A1 (GND), J4.A12 (GND), J4.B1 (GND), J4.B12 (GND), J4.S1 (SHIELD), J9.2, Q1.3, Q2.3, R10.2, R14.1, R9.2, U2.5 (GND), U4.10 (GND_1), U4.11 (GND_2), U4.22 (GND_3), U4.23 (GND_4), U4.35 (GND_5), U4.36 (GND_6), U4.4 (AGND_1), U4.41 (AGND_3), U4.42 (TEST), U4.47 (GND_7), U4.48 (GND_8), U4.49 (THERMAL_PAD), U4.9 (AGND_2)
- net LEFT_SCL: now also J2.A8, J2.B8, J2.C8, J2.D8, J2.E8, J2.F8, U3.5 (GPIO3); no longer U3.7 (GPIO5)
- net LEFT_SDA: now also J2.A6, J2.B6, J2.C6, J2.D6, J2.E6, J2.F6, U3.4 (GPIO2); no longer U3.6 (GPIO4)
- net LEFT_USB_DP: now also J1.A6 (D+), J1.B6 (D+)
- net RIGHT_SCL: now also J2.G8, J2.H8, J2.J8, J2.K8, J2.L8, J2.M8, U5.5 (GPIO3); no longer U5.7 (GPIO5)
- net RIGHT_SDA: now also J2.G6, J2.H6, J2.J6, J2.K6, J2.L6, J2.M6, U5.4 (GPIO2); no longer U5.6 (GPIO4)
- net POWER_SWITCH_LEFT: now reaches U3.27 (GPIO16)
- net POWER_SWITCH_LEFT: now also R46.1
- net at R35.1: now also U5.6 (GPIO4); no longer U5.15 (GPIO12)
- net TP_GND_LEFT: now reaches J2.A1
- net TP_GND_LEFT: now also J2.A3, J2.B1, J2.B3, J2.C1, J2.C3, J2.D1, J2.D3, J2.E1, J2.E3, J2.F1, J2.F3, Q1.2
- net TPL1_RL: now reaches J2.A11 (A_GREEN_2)
- net TPL1_RL: now also R16.2
- net TPL1_LED_OUT: now reaches J2.A2
- net TPL1_LED_OUT: now also J2.M4
- net TPL1_LED_IN: now reaches J2.A4
- net TPL1_LED_IN: now also J2.B2
- net TP_VCC_LEFT: now reaches J2.A5
- net TP_VCC_LEFT: now also J2.A7, J2.B5, J2.B7, J2.C5, J2.C7, J2.D5, J2.D7, J2.E5, J2.E7, J2.F5, J2.F7, J9.1
- net TPL1_LL: now reaches J2.A9 (A_GREEN_1)
- net TPL2_RL: now reaches J2.B11 (A_GREEN_4)
- net TPL2_RL: now also R18.2
- net TPL2_LED_IN: now reaches J2.B4
- net TPL2_LED_IN: now also J2.C2
- net TPL2_LL: now reaches J2.B9 (A_GREEN_3)
- net TPL2_LL: now also R17.2
- net TPL3_RL: now reaches J2.C11 (A_GREEN_6)
- net TPL3_RL: now also R20.2
- net TPL3_LED_IN: now reaches J2.C4
- net TPL3_LED_IN: now also J2.D2
- net TPL3_LL: now reaches J2.C9 (A_GREEN_5)
- net TPL3_LL: now also R19.2
- net TPL4_RL: now reaches J2.D11 (A_GREEN_8)
- net TPL4_RL: now also R22.2
- net TPL4_LED_IN: now reaches J2.D4
- net TPL4_LED_IN: now also J2.E2
- net TPL4_LL: now reaches J2.D9 (A_GREEN_7)
- net TPL4_LL: now also R21.2
- net TPL5_RL: now reaches J2.E11 (A_GREEN_10)
- net TPL5_RL: now also R24.2
- net TPL5_LED_IN: now reaches J2.E4
- net TPL5_LED_IN: now also J2.F2
- net TPL5_LL: now reaches J2.E9 (A_GREEN_9)
- net TPL5_LL: now also R23.2
- net TPL6_RL: now reaches J2.F11 (A_GREEN_12)
- net TPL6_RL: now also R26.2
- net TPL6_LED_IN: now reaches J2.F4
- net TPL6_LED_IN: now also J7.1 (Pin_1), J7.2 (Pin_2), J7.3 (Pin_3), J7.4 (Pin_4)
- net TPL6_LL: now reaches J2.F9 (A_GREEN_11)
- net TPL6_LL: now also R25.2
- net TP_GND_RIGHT: now reaches J2.G1
- net TP_GND_RIGHT: now also J2.G3, J2.H1, J2.H3, J2.J1, J2.J3, J2.K1, J2.K3, J2.L1, J2.L3, J2.M1, J2.M3, Q2.2
- net TPR6_LL: now reaches J2.G10 (A_GREEN_13)
- net TPR6_LL: now also R44.2
- net TPR6_RL: now reaches J2.G12 (A_GREEN_14)
- net TPR6_RL: now also R45.2
- net TPR6_LED_OUT: now reaches J2.G2
- net TPR5_LED_OUT: now reaches J2.G4
- net TPR5_LED_OUT: now also J2.H2
- net TP_VCC_RIGHT: now reaches J2.G5
- net TP_VCC_RIGHT: now also J2.G7, J2.H5, J2.H7, J2.J5, J2.J7, J2.K5, J2.K7, J2.L5, J2.L7, J2.M5, J2.M7, J10.1
- net TPR5_LL: now reaches J2.H10 (A_GREEN_15)
- net TPR5_LL: now also R42.2
- net TPR5_RL: now reaches J2.H12 (A_GREEN_16)
- net TPR5_RL: now also R43.2
- net TPR4_LED_OUT: now reaches J2.H4
- net TPR4_LED_OUT: now also J2.J2
- net TPR4_LL: now reaches J2.J10 (A_GREEN_17)
- net TPR4_LL: now also R40.2
- net TPR4_RL: now reaches J2.J12 (A_GREEN_18)
- net TPR4_RL: now also R41.2
- net TPR3_LED_OUT: now reaches J2.J4
- net TPR3_LED_OUT: now also J2.K2
- net TPR3_LL: now reaches J2.K10 (A_GREEN_19)
- net TPR3_LL: now also R38.2
- net TPR3_RL: now reaches J2.K12 (A_GREEN_20)
- net TPR3_RL: now also R39.2
- net TPR2_LED_OUT: now reaches J2.K4
- net TPR2_LED_OUT: now also J2.L2
- net TPR2_LL: now reaches J2.L10 (A_GREEN_21)
- net TPR2_LL: now also R36.2
- net TPR2_RL: now reaches J2.L12 (A_GREEN_22)
- net TPR2_RL: now also R37.2
- net TPR1_LED_OUT: now reaches J2.L4
- net TPR1_LED_OUT: now also J2.M2
- net TPR1_LL: now reaches J2.M10 (A_GREEN_23)
- net TPR1_RL: now reaches J2.M12 (A_GREEN_24)
- net at U5.16 (GPIO13): now also R42.1
- net at U3.11 (GPIO8): now also R20.1
- net at U3.12 (GPIO9): now also R19.1
- net at U3.13 (GPIO10): now also R22.1
- net at U3.14 (GPIO11): now also R21.1; no longer R15.1
- net at U3.15 (GPIO12): now also R24.1
- net at U3.16 (GPIO13): now also R23.1
- net at U3.17 (GPIO14): now also R26.1
- net at U3.18 (GPIO15): now also R25.1
- net at U3.8 (GPIO6): now also R18.1
- net at U3.9 (GPIO7): now also R17.1
- net VRAW: now reaches C1.2, D2.1 (K), D3.1 (K), U1.3 (VI)
- net VRAW: now also D1.1 (K), U4.40 (VREGIN)
- net at U5.17 (GPIO14): now also R45.1
- net at U5.18 (GPIO15): now also R44.1
- net at U5.11 (GPIO8): now also R39.1
- net at U5.12 (GPIO9): now also R38.1
- net at U5.13 (GPIO10): now also R41.1
- net at U5.14 (GPIO11): now also R40.1; no longer R34.1
- net POWER_SWITCH_RIGHT: now reaches U5.27 (GPIO16)
- net POWER_SWITCH_RIGHT: now also R47.1
- net at U5.8 (GPIO6): now also R37.1
- net at U5.9 (GPIO7): now also R36.1
- net LEFT_USB_DM renamed LEFT_USB_DN
- net RIGHT_USB_DM renamed RIGHT_USB_DN
- new net: Q2.1, R47.2
- new net: J4.B5 (CC2), R10.1
- new net: R43.1, U5.15 (GPIO12)
- new net: C13.1, U4.38 (VCCCORE)
- new net: R16.1, U3.6 (GPIO4)
- new net: R15.1, U3.7 (GPIO5)
- new net: Q1.1, R46.2
- new net: R14.2, U4.5 (REF)
- new net: R8.1, U2.4 (DO)
- new net: R34.1, U5.7 (GPIO5)
- new net: J4.A5 (CC1), R9.1
- new net: C19.2, U4.37 (VCCA)
- new net: R12.2, U4.34 (~{RESET})
- new net LED_EEPROM_CS: U2.1 (CS), U4.45 (EECS)
- new net LED_EEPROM_DATA: R8.2, U2.3 (DI), U4.43 (EEDATA)
- new net LED_EEPROM_SCLK: U2.2 (SCLK), U4.44 (EECLK)
- new net LED_GP0: J8.4 (Pin_4), U4.17 (ADBUS4)
- new net LED_GP1: J8.3 (Pin_3), U4.18 (ADBUS5)
- new net LED_GP2: J8.2 (Pin_2), U4.19 (ADBUS6)
- new net LED_GP3: J8.1 (Pin_1), U4.20 (ADBUS7)
- new net LED_TCK: J8.8 (Pin_8), U4.13 (ADBUS0)
- new net LED_TDI: J8.7 (Pin_7), U4.14 (ADBUS1)
- new net LED_TDO: J8.6 (Pin_6), U4.15 (ADBUS2)
- new net LED_TMS: J8.5 (Pin_5), U4.16 (ADBUS3)
- new net LED_USB_DN: J4.A7 (D-), J4.B7 (D-), U4.6 (DM)
- new net LED_USB_DP: J4.A6 (D+), J4.B6 (D+), U4.7 (DP)
- new net LED_USB_VBUS: D1.2 (A), J4.A4 (VBUS), J4.A9 (VBUS), J4.B4 (VBUS), J4.B9 (VBUS)
- new net LED_VCC: C23.1, C24.1, R12.1, U2.8 (VCC), U4.12 (VCCIO_1), U4.24 (VCCIO_2), U4.3 (VPHY), U4.39 (VCCD), U4.46 (VCCIO_3), U4.8 (VPLL)
- new net LED_XIN: C30.2, U4.1 (XCSI), Y3.1
- new net LED_XOUT: C31.2, U4.2 (XCSO), Y3.2
- no-connect marks 6 -> 49
Other:
- moved on the sheet: C1, C10, C16, C2, C20, C26, C27, C28, C3, C34, C37, C39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

Commit message: A few changes that needed to be pushed, the power switching circuitry has been removed temporarily to allow for manual power switching. I also baked the FT232HQ connection to the LED bus and changed the Via sizes to match the drilling specs required by most PCB fab services.
Parts:
- removed J7: Conn_02x02_Odd_Even, Connector_PinHeader_2.54mm:PinHeader_2x02_P2.54mm_Vertical, symbol Connector_Generic:Conn_02x02_Odd_Even
- removed J8: Conn_01x08_Male, Connector_PinHeader_2.54mm:PinHeader_1x08_P2.54mm_Vertical, symbol Connector:Conn_01x08_Male
- removed Q1, Q2: IRLB8721PBF, SamacSys_Parts:TO254P483X1016X1994-3P, symbol SamacSys_Parts:IRLB8721PBF
- removed R46, R47: 275, Resistor_SMD:R_0402_1005Metric, symbol Device:R_US
Connections:
- net LED_TDI is gone; now on net TPL6_LED_IN: U4.14 (ADBUS1)
- net TP_GND_LEFT is gone; now on net Earth: J2.A1, J2.A3, J2.B1, J2.B3, J2.C1, J2.C3, J2.D1, J2.D3, J2.E1, J2.E3, J2.F1, J2.F3
- net TP_GND_RIGHT is gone; now on net Earth: J2.G1, J2.G3, J2.H1, J2.H3, J2.J1, J2.J3, J2.K1, J2.K3, J2.L1, J2.L3, J2.M1, J2.M3
- net LED_GP0: no longer names the net of U4.17 (ADBUS4)
- net LED_GP1: no longer names the net of U4.18 (ADBUS5)
- net LED_GP2: no longer names the net of U4.19 (ADBUS6)
- net LED_GP3: no longer names the net of U4.20 (ADBUS7)
- net LED_TCK: no longer names the net of U4.13 (ADBUS0)
- net LED_TDO: no longer names the net of U4.15 (ADBUS2)
- net LED_TMS: no longer names the net of U4.16 (ADBUS3)
- net POWER_SWITCH_LEFT: no longer names the net of U3.27 (GPIO16)
- net POWER_SWITCH_RIGHT: no longer names the net of U5.27 (GPIO16)
- no-connect marks 49 -> 58
Other:
- moved on the sheet: J10
